Commit message: 実機に対応

File: er_crane_x7_description/urdf/crane_x7.urdf.xacro (robot description, xacro)
@@ -11,4 +11,7 @@
   <xacro:include filename="$(find er_crane_x7_description)/urdf/crane_x7.gazebo.xacro"/>
   <xacro:include filename="$(find crane_x7_description)/urdf/crane_x7.gazebo_ros2_control.xacro"/>
+  <xacro:macro name="er_crane_x7 "/>
+  <xacro:arg name="parent_link" default="base_link" />
+  <xacro:arg name="gen_link" default="" />
   <xacro:arg name="use_gazebo" default="false" />
   <xacro:arg name="use_d435" default="false" />
@@ -20,12 +23,4 @@
   <xacro:arg name="gz_control_config_package" default="" />
   <xacro:arg name="gz_control_config_file_path" default="" />
-  <!-- Link to provide the location reference for the arm -->
-  <link name="base_link"/>
-  <!-- Used for fixing robot to Gazebo 'base_link' -->
-  <link name="world"/>
-  <joint name="base_link_to_world_joint" type="fixed">
-    <parent link="world"/>
-    <child link="base_link"/>
-  </joint>
   <xacro:property name="M_PI" value="3.14159"/>
   <!-- D435 camera name -->
@@ -100,4 +95,7 @@
   <xacro:property name="JOINT_HAND_LOWER_LIMIT" value="${radians(-5)}"/>
   <xacro:property name="JOINT_HAND_UPPER_LIMIT" value="${radians(90)}"/>
+  <xacro:if value="$(arg gen_link)">
+    <link name="base_link"/>
+  </xacro:if>
   <!-- Use the crane_x7 macro to configure a Crane X7 arm with desired joint
        velocities limit and lower/upper limits for the first joint. This
@@ -105,5 +103,5 @@
        right-handed robots. -->
   <xacro:crane_x7
-    parent="base_link"
+    parent="$(arg parent_link)"
     name_link_mounting_plate="${NAME_LINK_MOUNTING_PLATE}"
     name_link_base="${NAME_LINK_BASE}"

File: er_crane_x7_description/urdf/crane_x7.xacro (robot description, xacro)
@@ -3,5 +3,5 @@
   <xacro:include filename="$(find crane_x7_description)/urdf/crane_x7_arm.xacro"/>
   <xacro:include filename="$(find crane_x7_description)/urdf/crane_x7_mounting_plate.xacro"/>
-  <xacro:include filename="$(find crane_x7_description)/urdf/crane_x7_wide_two_finger_gripper.xacro"/>
+  <xacro:include filename="$(find er_crane_x7_description)/urdf/crane_x7_wide_two_finger_gripper.xacro"/>
   <xacro:include filename="$(find crane_x7_description)/urdf/crane_x7_rt_logos.xacro"/>
   <material name="black">
@@ -178,4 +178,5 @@
     <!-- End effector -->
     <xacro:crane_x7_wide_two_finger_gripper
+        parent_link="${parent}"
         name_link_gripper_base="${name_link_gripper_base}"
         name_link_gripper_finger_a="${name_link_gripper_finger_a}"
