Commit message: modifired for erkachaka

File: er_crane_x7_description/urdf/crane_x7_wide_two_finger_gripper.xacro (robot description, xacro)
@@ -75,5 +75,5 @@
     -->
     <joint name="${name_joint_gripper_finger_b}_mimic" type="fixed">
-      <parent link="${parent_link}" />
+      <parent link="${name_link_gripper_base}" />
       <child link="dummy_mimic_fix" />
     </joint>
